File: LED Dimmer Board.sch (KiCad schematic (older format))
At the start: 10 parts, among them CON1 BARREL_JACK, U1 555

Commit message: Add files via upload
Parts:
- C1, C2: footprint (none) -> Capacitors_ThroughHole:C_Rect_L7_W2_P5
- R1, R2: footprint (none) -> Resistors_ThroughHole:Resistor_Horizontal_RM7mm
- RV1: footprint (none) -> Potentiometers:Potentiometer_WirePads_Small
- U1: footprint (none) -> Housings_DIP:DIP-8_W7.62mm
Other:
- note added: "LED: 20-30 mA\n 3.2-3.6 Vf\n 2330 mcd\nR1: 100 Ohm\nR2: 90 Ohm\nD1, D2: 1N4148 (or 1N914)\nCON1: 2.1 mm DC Barrel Jack\nC1, C2: 100 nF\nPOT: 10k\n"
- note added: "Warm White (3000 K) LED Circuit"
- note removed: "LED: 20-30 mA; 3.2-3.6 Vf; 2330 mcd\nR1: 100 Ohm\nR2: 90 Ohm\nD1, D2: 1N4148\nCON1: 2.1 mm DC Barrel Jack\nC1, C2: 100 nF\nPOT: 10k\n"
- note removed: "Warm White LED Circuit"
Changed lines of the file:
@@
 F 0 "U1" H 6730 2485 60  0000 C CNN
 F 1 "555" H 6105 3185 60  0000 C CNN
-F 2 "" H 6155 2835 60  0001 C CNN
+F 2 "Housings_DIP:DIP-8_W7.62mm" H 6155 2835 60  0001 C CNN
 F 3 "" H 6155 2835 60  0001 C CNN
 	1    6080 3260
@@
 F 0 "D3" H 7080 4110 50  0000 C CNN
 F 1 "LED" H 7080 3910 50  0000 C CNN
-F 2 "" H 7080 4010 50  0000 C CNN
+F 2 "" H 7080 4010 50  0001 C CNN
 F 3 "" H 7080 4010 50  0000 C CNN
 	1    7080 4010
@@
 F 0 "RV1" H 4605 3380 50  0000 C CNN
 F 1 "10k" H 4605 3460 50  0000 C CNN
-F 2 "" H 4605 3460 50  0000 C CNN
+F 2 "Potentiometers:Potentiometer_WirePads_Small" H 4605 3460 50  0001 C CNN
 F 3 "" H 4605 3460 50  0000 C CNN
 	1    4605 3460
@@
 F 0 "R1" V 4925 2655 50  0000 C CNN
 F 1 "100" V 4845 2655 50  0000 C CNN
-F 2 "" V 4775 2655 50  0000 C CNN
+F 2 "Resistors_ThroughHole:Resistor_Horizontal_RM7mm" V 4775 2655 50  0001 C CNN
 F 3 "" H 4845 2655 50  0000 C CNN
 	1    4845 2655
@@
 F 0 "R2" V 7160 3405 50  0000 C CNN
 F 1 "90" V 7080 3405 50  0000 C CNN
-F 2 "" V 7010 3405 50  0000 C CNN
+F 2 "Resistors_ThroughHole:Resistor_Horizontal_RM7mm" V 7010 3405 50  0001 C CNN
 F 3 "" H 7080 3405 50  0000 C CNN
 	1    7080 3405
@@
 F 0 "C2" H 6430 4740 50  0000 L CNN
 F 1 "100nF" H 6430 4540 50  0000 L CNN
-F 2 "" H 6443 4490 50  0000 C CNN
+F 2 "Capacitors_ThroughHole:C_Rect_L7_W2_P5" H 6443 4490 50  0001 C CNN
 F 3 "" H 6405 4640 50  0000 C CNN
 	1    6405 4640
@@
 F 0 "C1" H 5085 4300 50  0000 L CNN
 F 1 "100nF" H 5085 4100 50  0000 L CNN
-F 2 "" H 5098 4050 50  0000 C CNN
+F 2 "Capacitors_ThroughHole:C_Rect_L7_W2_P5" H 5098 4050 50  0001 C CNN
 F 3 "" H 5060 4200 50  0000 C CNN
 	1    5060 4200
@@
 F 0 "D2" H 4845 3260 50  0000 C CNN
 F 1 "1N4148" H 4845 3060 40  0000 C CNN
-F 2 "" H 4845 3160 50  0000 C CNN
+F 2 "" H 4845 3160 50  0001 C CNN
 F 3 "" H 4845 3160 50  0000 C CNN
 	1    4845 3160
@@
 F 0 "D1" H 4360 3260 50  0000 C CNN
 F 1 "1N4148" H 4360 3060 40  0000 C CNN
-F 2 "" H 4360 3160 50  0000 C CNN
+F 2 "" H 4360 3160 50  0001 C CNN
 F 3 "" H 4360 3160 50  0000 C CNN
 	1    4360 3160
@@
 F 0 "CON1" H 4600 1775 50  0000 C CNN
 F 1 "BARREL_JACK" H 4600 1325 50  0000 C CNN
-F 2 "" H 4600 1525 50  0000 C CNN
+F 2 "" H 4600 1525 50  0001 C CNN
 F 3 "" H 4600 1525 50  0000 C CNN
 	1    4600 1525
@@
 	1880 3475 1880 1620
 Text Notes 1955 1730 0    60   ~ 0
-Warm White LED Circuit
-Text Notes 1935 2400 0    45   ~ 0
-LED:  20-30 mA; 3.2-3.6 Vf; 2330 mcd\nR1:  100 Ohm\nR2:  90 Ohm\nD1, D2:  1N4148\nCON1:  2.1 mm DC Barrel Jack\nC1, C2:  100 nF\nPOT:  10k\n
+Warm White (3000 K) LED Circuit
+Text Notes 1925 2590 0    45   ~ 0
+LED:  20-30 mA\n      3.2-3.6 Vf\n      2330 mcd\nR1:  100 Ohm\nR2:  90 Ohm\nD1, D2:  1N4148 (or 1N914)\nCON1:  2.1 mm DC Barrel Jack\nC1, C2:  100 nF\nPOT:  10k\n
 $EndSCHEMATC
